File: Sensor_board.kicad_sch (KiCad schematic)
At the start: 86 parts, among them IC1 STM32G491CET6, J1 Conn_01x04, J10 Conn_01x05, J11 Conn_02x07_Odd_Even, J12 Conn_01x04, J13 Conn_01x02, J14 Conn_01x02, J15 Conn_01x02, J16 Conn_01x02, J2 Conn_01x04, J3 Conn_01x02, J4 Conn_01x04, J5 Conn_01x04, J6 Conn_01x02, J7 Conn_01x04, J8 Conn_01x04, J9 Conn_01x04, SW1 SW_Push, SW2 SW_Push, U1 SN65HVD230, U2 DIO6913, U3 SN65HVD230, U4 L78L33_SOT89, Y1 Crystal

Commit message: changed mcu pinout
Parts:
- removed J13, J14, J15: Conn_01x02, symbol Connector_Generic:Conn_01x02
- removed J8: Conn_01x04, symbol Connector_Generic:Conn_01x04
- added IC2: STM32G491CET6, STM32G491CET6:QFP50P900X900X160-48N, symbol STM32G491CET6:STM32G491CET6
- added J13, J17, J19: Conn_01x04, symbol Connector_Generic:Conn_01x04
- added J14, J15, J8: Conn_01x06, symbol Connector_Generic:Conn_01x06
- added J18: Conn_01x02, symbol Connector_Generic:Conn_01x02
- added J20: Conn_01x03, symbol Connector_Generic:Conn_01x03
- added R17, R18, R19, R20: 10k, Resistor_SMD:R_0603_1608Metric, symbol Device:R_Small
Connections:
- net PA8 is gone; now on net I2C_SDA: IC1.30 (PA8)
- net +3.3V: now also J4.1 (Pin_1), J7.1 (Pin_1), IC2.1 (VBAT), IC2.20 (VREF+), IC2.21 (VDDA), IC2.24 (VDD_1), IC2.36 (VDD_2), IC2.48 (VDD_3), J13.1 (Pin_1), J14.1 (Pin_1), J15.1 (Pin_1), J17.1 (Pin_1), J18.1 (Pin_1), J19.1 (Pin_1), J8.1 (Pin_1), R17.1, R18.1, R19.1, R20.1
- net +5V: now also J16.1 (Pin_1)
- net BOOT0: now also IC2.45 (PB8-BOOT0)
- net FDCAN1_RX: now also IC2.33 (PA11)
- net FDCAN1_TX: now also IC2.34 (PA12)
- net FDCAN2_RX: now also IC2.27 (PB13)
- net FDCAN2_TX: now also IC2.26 (PB12)
- net GND: now also J1.2 (Pin_2), J16.2 (Pin_2), J4.4 (Pin_4), J7.2 (Pin_2), IC2.19 (VSSA), IC2.23 (VSS_1), IC2.35 (VSS_2), IC2.47 (VSS_3), J13.4 (Pin_4), J14.2 (Pin_2), J15.2 (Pin_2), J17.2 (Pin_2), J18.2 (Pin_2), J19.4 (Pin_4), J8.2 (Pin_2)
- net I2C1_SCL: now also J7.3 (Pin_3), IC2.39 (PA15), R17.2
- net I2C1_SDA: now also J7.4 (Pin_4), IC2.44 (PB7), R18.2
- net I2C2_SCL: now also IC1.31 (PA9), IC2.31 (PA9), J17.3 (Pin_3), R20.2; no longer IC1.32 (PA10)
- net I2C_SDA: now also IC2.30 (PA8); no longer IC1.31 (PA9)
- net NRST: now also J1.4 (Pin_4), IC2.7 (PG10_-_NRST)
- net PB0: now also IC2.16 (PB0), J14.6 (Pin_6)
- net PB1: now also IC2.17 (PB1), J8.6 (Pin_6)
- net PB14: now also IC2.28 (PB14)
- net PB15: now also IC2.29 (PB15)
- net PB2: now also IC2.18 (PB2), J15.6 (Pin_6)
- net PB9: now also IC2.46 (PB9)
- net PC13: now also IC2.2 (PC13)
- net PC14: now also IC2.3 (PC14_-_OSC32_IN)
- net PC15: now also IC2.4 (PC15_-_OSC32_OUT)
- net RCC_OSC_IN: now also IC2.5 (PF0_-_OSC_IN)
- net RCC_OSC_OUT: now also IC2.6 (PF1_-_OSC_OUT)
- net SPI1_MISO: now also J14.4 (Pin_4)
- net SPI1_MOSI: now also IC2.15 (PA7), J14.5 (Pin_5)
- net SPI1_SCK: now also IC2.13 (PA5), J14.3 (Pin_3)
- net SWCLK: now also J1.1 (Pin_1), IC2.38 (PA14)
- net SWDIO: now also J1.3 (Pin_3), IC2.37 (PA13)
- net USART3_RX: now also IC2.25 (PB11)
- net USART3_TX: now also IC2.22 (PB10)
- net USART1_RX: now reaches J4.2 (Pin_2)
- net USART1_RX: now also IC1.32 (PA10), IC2.32 (PA10), J13.2 (Pin_2), J19.2 (Pin_2)
- net USART1_TX: now reaches J4.3 (Pin_3)
- net USART1_TX: now also IC1.43 (PB6), IC2.43 (PB6), J13.3 (Pin_3), J19.3 (Pin_3)
- net PB3 renamed SPI3_SCK
- net SPI3_SCK: now also IC2.40 (PB3), J15.3 (Pin_3)
- net PB4 renamed SPI3_MISO
- net SPI3_MISO: now also IC2.41 (PB4), J15.4 (Pin_4)
- net PB5 renamed SPI3_MOSI
- net SPI3_MOSI: now also IC2.42 (PB5), J15.5 (Pin_5)
- net TIM2_CH1 renamed ADC1_IN1
- net ADC1_IN1: now also IC2.8 (PA0)
- net TIM2_CH2 renamed ADC1_IN2
- net ADC1_IN2: now also IC1.10 (PA2), IC2.10 (PA2), IC2.9 (PA1)
- net USART2_RX renamed ADC1_IN3
- net ADC1_IN3: now also IC2.11 (PA3)
- removed net USART2_TX: IC1.10 (PA2), IC1.43 (PB6)
- new net I2C2_SDA: J17.4 (Pin_4), R19.2
- new net SPI2_MISO: J8.4 (Pin_4)
- new net SPI2_MOSI: J8.5 (Pin_5)
- new net SPI2_SCK: J8.3 (Pin_3)
- new net TIM3_CH1: IC2.14 (PA6)
- new net TIM3_CH2: IC2.12 (PA4)
Other:
- note added: "POWER"
- moved on the sheet: J1, J4, J7

Commit message: 50% of trace
Parts:
- removed D1: AMBER LED, LED_SMD:LED_0805_2012Metric, symbol Device:LED_Small
- removed D2: BLUE LED, LED_SMD:LED_0805_2012Metric, symbol Device:LED_Small
- removed IC1: STM32G491CET6, STM32G491CET6:QFP50P900X900X160-48N, symbol STM32G491CET6:STM32G491CET6
- removed J1, J12: Conn_01x04, symbol Connector_Generic:Conn_01x04
- removed J10: Conn_01x05, Connector_PinHeader_2.54mm:PinHeader_1x05_P2.54mm_Vertical, symbol Connector_Generic:Conn_01x05
- removed J11: Conn_02x07_Odd_Even, symbol Connector_Generic:Conn_02x07_Odd_Even
- removed J15: Conn_01x06, symbol Connector_Generic:Conn_01x06
- removed J9: Conn_01x04, Connector_PinHeader_2.54mm:PinHeader_1x04_P2.54mm_Vertical, symbol Connector_Generic:Conn_01x04
- removed JP4, JP5: SolderJumper_3_Bridged12, symbol Jumper:SolderJumper_3_Bridged12
- removed R4, R5: 1k, Resistor_SMD:R_0603_1608Metric, symbol Device:R_Small
- removed TP3, TP4, TP8, TP9: TestPoint, TestPoint:TestPoint_Pad_1.0x1.0mm, symbol Connector:TestPoint
- added D2, D3: ~, LED_SMD:LED_0805_2012Metric_Pad1.15x1.40mm_HandSolder, symbol Device:LED
- added H1, H2, H3, H4: MountingHole_Pad, MountingHole:MountingHole_3.2mm_M3_DIN965_Pad, symbol Mechanical:MountingHole_Pad
- added J12: Conn_01x02, Connector_Molex:Molex_SPOX_5267-02A_1x02_P2.50mm_Vertical, symbol Connector_Generic:Conn_01x02
- added J17: Conn_02x08_Odd_Even, Connector_PinHeader_2.54mm:PinHeader_2x08_P2.54mm_Vertical, symbol Connector_Generic:Conn_02x08_Odd_Even
- added J19, J20, J21, J22: Conn_01x03, Connector_Molex:Molex_SPOX_5267-03A_1x03_P2.50mm_Vertical, symbol Connector_Generic:Conn_01x03
- added J23, J24: Conn_01x04, easyeda2kicad:CONN-TH_4P-XT30PW-M, symbol Connector_Generic:Conn_01x04
- added J9: Conn_01x05, Connector_PinHeader_2.54mm:PinHeader_1x05_P2.54mm_Vertical, symbol Connector_Generic:Conn_01x05
- added JP1: Jumper_2_Open, Connector_PinHeader_2.54mm:PinHeader_1x02_P2.54mm_Vertical, symbol Jumper:Jumper_2_Open
- added R13, R14: 1k, Resistor_SMD:R_0603_1608Metric_Pad0.98x0.95mm_HandSolder, symbol Device:R_Small
- C1, C10, C19, C20, C21, C22, C23, C24, C25, C3, C8, C9: footprint Capacitor_SMD:C_0603_1608Metric -> Capacitor_SMD:C_0603_1608Metric_Pad1.08x0.95mm_HandSolder
- C11, C12, C14, C15: footprint Capacitor_SMD:C_0805_2012Metric -> Capacitor_SMD:C_0805_2012Metric_Pad1.18x1.45mm_HandSolder
- C13, C16, C6, C7: value 100n/50V -> 100n/50V; footprint Capacitor_SMD:C_0603_1608Metric -> Capacitor_SMD:C_0603_1608Metric_Pad1.08x0.95mm_HandSolder
- C17, C18: footprint Capacitor_SMD:C_0603_1608Metric -> Capacitor_SMD:C_0603_1608Metric_Pad1.08x0.95mm_HandSolder; now not fitted; now left out of the parts list
- C2, C4, C5: footprint Capacitor_SMD:C_1206_3216Metric -> Capacitor_SMD:C_1206_3216Metric_Pad1.33x1.80mm_HandSolder
- D4, D5, D6: footprint LED_SMD:LED_0805_2012Metric -> LED_SMD:LED_0805_2012Metric_Pad1.15x1.40mm_HandSolder
- IC1: renamed from IC2; footprint STM32G491CET6:QFP50P900X900X160-48N -> Package_QFP:LQFP-48_7x7mm_P0.5mm
- J10: renamed from J16; footprint (none) -> Connector_Molex:Molex_SPOX_5267-02A_1x02_P2.50mm_Vertical
- J11: renamed from J18; footprint (none) -> Connector_Molex:Molex_SPOX_5267-02A_1x02_P2.50mm_Vertical
- J13: renamed from J7; footprint (none) -> Connector_Molex:Molex_SPOX_5267-04A_1x04_P2.50mm_Vertical
- J14: renamed from J17; footprint (none) -> Connector_Molex:Molex_SPOX_5267-04A_1x04_P2.50mm_Vertical
- J15: renamed from J14; footprint (none) -> Connector_Molex:Molex_SPOX_5267-06A_1x06_P2.50mm_Vertical
- J16: renamed from J8; footprint (none) -> Connector_Molex:Molex_SPOX_5267-06A_1x06_P2.50mm_Vertical
- J18: renamed from J20; footprint (none) -> Connector_Molex:Molex_SPOX_5267-03A_1x03_P2.50mm_Vertical
- J2: footprint (none) -> easyeda2kicad:CONN-TH_4P-XT30PW-M
- J3: footprint (none) -> Connector_Molex:Molex_SPOX_5267-02A_1x02_P2.50mm_Vertical
- J4: footprint (none) -> Connector_Molex:Molex_SPOX_5267-04A_1x04_P2.50mm_Vertical
- J5: renamed from J13; footprint (none) -> Connector_Molex:Molex_SPOX_5267-04A_1x04_P2.50mm_Vertical
- J6: renamed from J19; footprint (none) -> Connector_Molex:Molex_SPOX_5267-04A_1x04_P2.50mm_Vertical; now not fitted; now left out of the parts list
- J7: renamed from J5; footprint (none) -> easyeda2kicad:CONN-TH_4P-XT30PW-M
- J8: renamed from J6; footprint (none) -> Connector_Molex:Molex_SPOX_5267-02A_1x02_P2.50mm_Vertical
- JP2: renamed from JP1; footprint Jumper:SolderJumper-3_P1.3mm_Open_Pad1.0x1.5mm_NumberLabels -> Jumper:SolderJumper-3_P1.3mm_Open_Pad1.0x1.5mm
- JP3: renamed from JP2; footprint Jumper:SolderJumper-3_P1.3mm_Open_Pad1.0x1.5mm_NumberLabels -> Jumper:SolderJumper-3_P1.3mm_Open_Pad1.0x1.5mm
- JP4: renamed from JP3; footprint (none) -> Jumper:SolderJumper-2_P1.3mm_Open_RoundedPad1.0x1.5mm
- R1: footprint Resistor_SMD:R_0603_1608Metric -> Resistor_SMD:R_0603_1608Metric_Pad0.98x0.95mm_HandSolder; MPN WF06P-100K-5% -> WF06P-10K-5%
- R10: renamed from R20; footprint Resistor_SMD:R_0603_1608Metric -> Resistor_SMD:R_0603_1608Metric_Pad0.98x0.95mm_HandSolder
- R11: renamed from R9; footprint Resistor_SMD:R_0603_1608Metric -> Resistor_SMD:R_0603_1608Metric_Pad0.98x0.95mm_HandSolder
- R12: renamed from R10; footprint Resistor_SMD:R_0603_1608Metric -> Resistor_SMD:R_0603_1608Metric_Pad0.98x0.95mm_HandSolder
- R15: renamed from R11; footprint Resistor_SMD:R_0603_1608Metric -> Resistor_SMD:R_0603_1608Metric_Pad0.98x0.95mm_HandSolder
- R16: renamed from R12; footprint Resistor_SMD:R_0603_1608Metric -> Resistor_SMD:R_0603_1608Metric_Pad0.98x0.95mm_HandSolder
- R18: renamed from R14; footprint Resistor_SMD:R_0603_1608Metric -> Resistor_SMD:R_0603_1608Metric_Pad0.98x0.95mm_HandSolder
- R19: renamed from R15; footprint Resistor_SMD:R_0603_1608Metric -> Resistor_SMD:R_0603_1608Metric_Pad0.98x0.95mm_HandSolder
- R2, R3: footprint Resistor_SMD:R_0603_1608Metric -> Resistor_SMD:R_0603_1608Metric_Pad0.98x0.95mm_HandSolder
- R20: renamed from R16; footprint Resistor_SMD:R_0603_1608Metric -> Resistor_SMD:R_0603_1608Metric_Pad0.98x0.95mm_HandSolder
- R4: renamed from R6; footprint Resistor_SMD:R_0603_1608Metric -> Resistor_SMD:R_0603_1608Metric_Pad0.98x0.95mm_HandSolder
- R6: renamed from R18; footprint Resistor_SMD:R_0603_1608Metric -> Resistor_SMD:R_0603_1608Metric_Pad0.98x0.95mm_HandSolder
- R7: renamed from R19; footprint Resistor_SMD:R_0603_1608Metric -> Resistor_SMD:R_0603_1608Metric_Pad0.98x0.95mm_HandSolder
- R8: value 100k -> 10k; footprint Resistor_SMD:R_0603_1608Metric -> Resistor_SMD:R_0603_1608Metric_Pad0.98x0.95mm_HandSolder; MPN WF06P-100K-5% -> WF06P-10K-5%
- R9: renamed from R17; footprint Resistor_SMD:R_0603_1608Metric -> Resistor_SMD:R_0603_1608Metric_Pad0.98x0.95mm_HandSolder
- SW1: footprint robocik-footprints:SW_Push_1P1T_NO_CK_PTS647_Sx -> Button_Switch_THT:SW_PUSH_6mm; DSC USER BUTTON -> (none); MPN PTS647SK70SMTR2LFS -> (none); STORE https://www.mouser.pl/ProductDetail/CK/PTS647SK70SMTR2LFS?q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 -> (none); now not fitted; now left out of the parts list
- SW2: footprint robocik-footprints:SW_Push_1P1T_NO_CK_PTS647_Sx -> Button_Switch_THT:SW_PUSH_6mm; DSC BOOTLOADER -> (none); MPN PTS647SK70SMTR2LFS -> (none); STORE https://www.mouser.pl/ProductDetail/CK/PTS647SK70SMTR2LFS?q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 -> (none)
- TP5: footprint (none) -> TestPoint:TestPoint_Pad_1.0x1.0mm
- U2: footprint Package_TO_SOT_SMD:TSOT-23-6 -> Package_TO_SOT_SMD:TSOT-23-6_HandSoldering
- U4: footprint Package_TO_SOT_SMD:SOT-89-3 -> Package_TO_SOT_SMD:SOT-89-3_Handsoldering
- Y1: footprint (none) -> Crystal:Crystal_SMD_FOX_FE-2Pin_7.5x5.0mm_HandSoldering; now not fitted; now left out of the parts list
- renumbered D3 to D1, R13 to R17, R7 to R5
Connections:
- net CAN_1_RX is gone; now on net FDCAN1_RX: U1.4 (R)
- net CAN_1_TX is gone; now on net FDCAN1_TX: U1.1 (D)
- net CAN_2_RX is gone; now on net FDCAN2_RX: U3.4 (R)
- net CAN_2_TX is gone; now on net FDCAN2_TX: U3.1 (D)
- net I2C_SDA is gone; now on net I2C2_SDA: IC1.30 (PA8)
- net PB14 is gone; now on net SPI2_MISO: IC1.28 (PB14)
- net PB15 is gone; now on net SPI2_MOSI: IC1.29 (PB15)
- net SPI2_SCK is gone; now on net FDCAN2_RX: J16.3 (Pin_3)
- net SPI3_MISO is gone; now on net SPI1_MISO: IC1.41 (PB4)
- net SPI3_SCK is gone; now on net TIM2_CH2: IC1.40 (PB3)
- net TIM3_CH2 is gone; now on net PA4: IC1.12 (PA4)
- net UserButton is gone; now on net BOOT0: R1.1, SW1.1
- net +3.3V: now also J17.2 (Pin_2), J21.1 (Pin_1), J22.1 (Pin_1), J9.1 (Pin_1), JP1.1 (A)
- net +5V: now also J18.1 (Pin_1), J17.4 (Pin_4), J19.1 (Pin_1), J20.1 (Pin_1); no longer TP5.1
- net ADC1_IN1: now also J17.10 (Pin_10)
- net ADC1_IN2: now also J17.12 (Pin_12); no longer IC1.10 (PA2)
- net BOOT0: now also JP1.2 (B); no longer R8.1, SW2.1
- net CAN_1_H: now also J23.3 (Pin_3), J24.3 (Pin_3)
- net CAN_1_L: now also J23.4 (Pin_4), J24.4 (Pin_4)
- net CAN_2_H: now also R17.1, U3.7 (CANH)
- net CAN_2_L: now also R17.2, U3.6 (CANL)
- net GND: now also J18.3 (Pin_3), D2.1 (K), D3.1 (K), H1.1, H2.1, H3.1, H4.1, J12.2 (Pin_2), J17.1 (Pin_1), J17.3 (Pin_3), J19.3 (Pin_3), J20.3 (Pin_3), J21.3 (Pin_3), J22.3 (Pin_3), J23.2 (Pin_2), J24.2 (Pin_2), J9.3 (Pin_3)
- net NRST: now also J9.5 (Pin_5)
- net PA4: now also J17.14 (Pin_14), J22.2 (Pin_2)
- net PB0: now also J17.5 (Pin_5)
- net PB1: now also J17.7 (Pin_7)
- net PB2: now also J17.9 (Pin_9)
- net PB9: now also J17.13 (Pin_13)
- net PC13: now also R8.1, SW2.1, J17.15 (Pin_15)
- net PC14: now also J17.6 (Pin_6), R14.1
- net PC15: now also J17.8 (Pin_8), R13.1
- net SWCLK: now also J9.2 (Pin_2)
- net SWDIO: now also J9.4 (Pin_4)
- net USART1_RX: no longer J5.2 (Pin_2)
- net USART1_TX: no longer J5.3 (Pin_3)
- net VCC: now also J12.1 (Pin_1), J23.1 (Pin_1), J24.1 (Pin_1)
- net at C11.1, C12.1, C13.2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: now also TP5.1
- net TIM2_CH2: now reaches J18.2 (Pin_2)
- net ADC1_IN3 renamed USART2_RX
- net USART2_RX: now also J5.2 (Pin_2)
- net SPI3_MOSI renamed PB5
- net PB5: now also J17.11 (Pin_11)
- net TIM3_CH1 renamed PA6
- net PA6: now also J17.16 (Pin_16), J21.2 (Pin_2)
- net USART3_RX renamed TIM2_CH4
- net TIM2_CH4: now also J20.2 (Pin_2)
- net USART3_TX renamed TIM2_CH3
- net TIM2_CH3: now also J19.2 (Pin_2)
- new net: D2.2 (A), R13.2
- new net: D3.2 (A), R14.2
- new net USART2_TX: IC1.10 (PA2), J5.3 (Pin_3)
Other:
- note added: "Leak sensor"
- note added: "PWM"
- note added: "Programming"
- note added: "User button & LEDs"
- note removed: "USER BUTTON"
- note removed: "USER LEDS"
- moved on the sheet: IC1, J18, TP5

Commit message: 60% of trace
Parts:
- D4, D5, D6, J23, R18, R19, R20: now not fitted; now left out of the parts list
Changed lines of the file:
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@@
 		(at 256.54 24.765 0)
 		(unit 1)
-		(exclude_from_sim no)
-		(in_bom yes)
-		(on_board yes)
-		(dnp no)
+		(exclude_from_sim yes)
+		(in_bom no)
+		(on_board no)
+		(dnp yes)
 		(fields_autoplaced yes)
 		(property "Reference" "R18"
@@
 		(at 256.54 32.385 90)
 		(unit 1)
-		(exclude_from_sim no)
-		(in_bom yes)
-		(on_board yes)
-		(dnp no)
+		(exclude_from_sim yes)
+		(in_bom no)
+		(on_board no)
+		(dnp yes)
 		(fields_autoplaced yes)
 		(property "Reference" "D4"
@@
 		(at 270.51 24.765 0)
 		(unit 1)
-		(exclude_from_sim no)
-		(in_bom yes)
-		(on_board yes)
-		(dnp no)
+		(exclude_from_sim yes)
+		(in_bom no)
+		(on_board no)
+		(dnp yes)
 		(fields_autoplaced yes)
 		(property "Reference" "R19"
@@
 		(at 270.51 32.385 90)
 		(unit 1)
-		(exclude_from_sim no)
-		(in_bom yes)
-		(on_board yes)
-		(dnp no)
+		(exclude_from_sim yes)
+		(in_bom no)
+		(on_board no)
+		(dnp yes)
 		(fields_autoplaced yes)
 		(property "Reference" "D5"
@@
 		(at 282.575 32.385 90)
 		(unit 1)
-		(exclude_from_sim no)
-		(in_bom yes)
-		(on_board yes)
-		(dnp no)
+		(exclude_from_sim yes)
+		(in_bom no)
+		(on_board no)
+		(dnp yes)
 		(fields_autoplaced yes)
 		(property "Reference" "D6"
@@
 		(at 282.575 24.765 0)
 		(unit 1)
-		(exclude_from_sim no)
-		(in_bom yes)
-		(on_board yes)
-		(dnp no)
+		(exclude_from_sim yes)
+		(in_bom no)
+		(on_board no)
+		(dnp yes)
 		(fields_autoplaced yes)
 		(property "Reference" "R20"
@@
 		(at 30.48 157.48 0)
 		(unit 1)
-		(exclude_from_sim no)
-		(in_bom yes)
-		(on_board yes)
-		(dnp no)
+		(exclude_from_sim yes)
+		(in_bom no)
+		(on_board no)
+		(dnp yes)
 		(fields_autoplaced yes)
 		(property "Reference" "J23"

Commit message: almost done
Parts:
- removed H1, H2, H3, H4: MountingHole_Pad, MountingHole:MountingHole_3.2mm_M3_DIN965_Pad, symbol Mechanical:MountingHole_Pad
- added H5, H6, H7, H8: MountingHole, MountingHole:MountingHole_3.2mm_M3_ISO7380, symbol Mechanical:MountingHole
- J10, J11, J12, J3, J8: now not fitted; now left out of the parts list
- JP4: footprint Jumper:SolderJumper-2_P1.3mm_Open_RoundedPad1.0x1.5mm -> Jumper:SolderJumper-2_P1.3mm_Open_TrianglePad1.0x1.5mm
Connections:
- net +3.3V: now also J17.4 (Pin_4); no longer J17.2 (Pin_2)
- net +5V: now also J17.2 (Pin_2); no longer J17.4 (Pin_4)

Commit message: major route chanses to improve overall layout
Parts:
- added JP5: SolderJumper_3_Open, Jumper:SolderJumper-3_P1.3mm_Open_Pad1.0x1.5mm, symbol Jumper:SolderJumper_3_Open
Connections:
- net +3.3V: now also JP5.1 (A)
- net +5V: now also JP5.3 (B); no longer J18.1 (Pin_1), J19.1 (Pin_1), J20.1 (Pin_1)
- net PB0: now also J16.6 (Pin_6), J17.13 (Pin_13); no longer J15.6 (Pin_6), J17.5 (Pin_5)
- net PB1: now also J15.6 (Pin_6), J17.11 (Pin_11); no longer J16.6 (Pin_6), J17.7 (Pin_7)
- net PB5: now also J17.7 (Pin_7); no longer J17.11 (Pin_11)
- net PB9: now also J17.5 (Pin_5); no longer J17.13 (Pin_13)
- new net: J18.1 (Pin_1), J19.1 (Pin_1), JP5.2 (C)
Other:
- moved on the sheet: J18, J19, J20

Commit message: final design version
Parts:
- added D7, D8: ~, LED_SMD:LED_0805_2012Metric_Pad1.15x1.40mm_HandSolder, symbol Device:LED
- added R21: 1k, Resistor_SMD:R_0603_1608Metric_Pad0.98x0.95mm_HandSolder, symbol Device:R_Small
- added R22: 120, Resistor_SMD:R_0603_1608Metric_Pad0.98x0.95mm_HandSolder, symbol Device:R_Small
- H5, H6, H7, H8: footprint MountingHole:MountingHole_3.2mm_M3_ISO7380 -> MountingHole:MountingHole_3.2mm_M3_ISO7380_Pad; now in the parts list
Connections:
- net +3.3V: now also R22.1
- net +5V: now also R21.1
- net GND: now also D7.1 (K), D8.1 (K)
- net at J20.1 (Pin_1): now also J18.1 (Pin_1), J19.1 (Pin_1), JP5.2 (C)
- new net: D7.2 (A), R21.2
- new net: D8.2 (A), R22.2
